File: Hardware/BuckConverter/senza-titolo.kicad_sch (KiCad schematic)
At the start: 1 part, among them U3 AD8411A

Commit message: Schematic V2 added board comunication connectors and decoupling C
Parts:
- removed U3: AD8411A, kicadLibFp:SOIC-8, symbol KicadLib:AD8411A
